File: piboard.brd (EAGLE design)
At the start: 131 x 151.9 mm, 79 parts, among them IC1 IS25LP256D-JLLE-TR, IC2 IS31FL3737-QFLS4-TR, U1 RP2040, Y1 ABLS-12.000MHZ-B4-T

Commit message: Daily check-in
Parts:
- removed Y1: ABLS-12.000MHZ-B4-T, ABLS-12.000MHZ-B4-T:XTAL_ABLS-12.000MHZ-B4-T
- added Q1: (no value), adafruit:NX3225
- moved RGB1 177.4 mm to (11.4, 78.7)
Connections:
- removed net XOUT_R: C21.1, R14.2, Y1.1
- new net G1: Q1.4
- new net G2: Q1.2
- new net SW01: RGB37.1, RGB38.1, RGB39.1, RGB40.1, RGB41.1, RGB42.1, RGB43.1, RGB44.1, RGB45.1, RGB46.1, RGB47.1, RGB48.1
- new net SW02: RGB37.3, RGB38.3, RGB39.3, RGB40.3, RGB41.3, RGB42.3, RGB43.3, RGB44.3, RGB45.3, RGB46.3, RGB47.3, RGB48.3
- new net SW03: RGB37.5, RGB38.5, RGB39.5, RGB40.5, RGB41.5, RGB42.5, RGB43.5, RGB44.5, RGB45.5, RGB46.5, RGB47.5, RGB48.5
- new net SW04: RGB25.1, RGB26.1, RGB27.1, RGB28.1, RGB29.1, RGB30.1, RGB31.1, RGB32.1, RGB33.1, RGB34.1, RGB35.1, RGB36.1
- new net SW05: RGB25.3, RGB26.3, RGB27.3, RGB28.3, RGB29.3, RGB30.3, RGB31.3, RGB32.3, RGB33.3, RGB34.3, RGB35.3, RGB36.3
- new net SW06: RGB25.5, RGB26.5, RGB27.5, RGB28.5, RGB29.5, RGB30.5, RGB31.5, RGB32.5, RGB33.5, RGB34.5, RGB35.5, RGB36.5
- new net SW07: RGB13.1, RGB14.1, RGB15.1, RGB16.1, RGB17.1, RGB18.1, RGB19.1, RGB20.1, RGB21.1, RGB22.1, RGB23.1, RGB24.1
- new net SW08: RGB13.3, RGB14.3, RGB15.3, RGB16.3, RGB17.3, RGB18.3, RGB19.3, RGB20.3, RGB21.3, RGB22.3, RGB23.3, RGB24.3
- new net SW09: RGB13.5, RGB14.5, RGB15.5, RGB16.5, RGB17.5, RGB18.5, RGB19.5, RGB20.5, RGB21.5, RGB22.5, RGB23.5, RGB24.5
- net GND: now also IC2.11, IC2.4, IC2.40, IC2.41
- net XIN: no longer Y1.2
Other:
- outline, holes or cut-outs redrawn

Commit message: update
Parts:
- added C13, C14, C22, C23, C25, C27, C29: 0.1uF, SparkFun-Capacitors:0402
- added C15, C16: 10uF, OPL_Capacitor:C0402
- added C17, C18: 4.7uF, OPL_Capacitor:C0402
- added C19, C24, C26, C28: 470nF 50V, OPL_Capacitor:C0402
- added C30, C31, C32, C33, C34, C35, C36, C37, C38, C39, C40, C41: 100nf, OPL_Capacitor:C0402
- added C42: 22uF, OPL_Capacitor:AVX-A
- added D1: BLUE-0402, OPL_Optoelectronics:LED-0402
- added D3: 20V-1A, OPL_Discrete_Semiconductor:SOD-123
- added D4: RED-0402, OPL_Optoelectronics:LED-0402
- added H1, H2, H3, H4, H5, H6, H7, H8: M25, M25:M25
- added J1: TYPE-C-31-M-12, TYPE-C-31-M-12:HRO_TYPE-C-31-M-12
- added J2: (no value), SparkFun-Connectors:JST-2-SMD
- added JP1: JUMPER-SMT_2_NO_SILK_ROUND, SparkFun-Jumpers:SMT-JUMPER_2_NO_SILK_ROUND
- added L2: 2.2nH, SparkFun-Coils:0402
- added LED1, LED10, LED11, LED12, LED2, LED3, LED4, LED5, LED6, LED7, LED8, LED9: WS2812B-2020, WS2812B-2020:WS2812B-2020
- added MK1: ICS-41350, ICS-41350:MIC_ICS-41350
- added Q2: 2.5A/30V/105mΩ, SparkFun-DiscreteSemi:SOT23-3
- added R11: 10k, SparkFun-Resistors:0603
- added R12: 470, SparkFun-Resistors:0402
- added R13: 2K, SparkFun-Resistors:0402
- added R15: 20K, SparkFun-Resistors:0402
- added R16, R17, R18: 100K, SparkFun-Resistors:0402
- added R19: 220, SparkFun-Resistors:0402
- added R3, R4, R7: 10K, SparkFun-Resistors:0402
- added R5, R6: 4.7K, SparkFun-Resistors:0402
- added R8, R9: 5.1K, SparkFun-Resistors:0402
- added S3: MOMENTARY-SWITCH-SPST-SMD-4.6X2.8MM, SparkFun-Switches:TACTILE_SWITCH_SMD_4.6X2.8MM
- added SW1: PCM12SMTR, PCM12SMTR:SW_PCM12SMTR
- added U2: BMI270, BMI270:XDCR_BMI270
- added U3: MIC5504-3.3YM5_TR, MIC5504-3.3YM5_TR:SOT95P280X145-5N
- added U4: MCP73831T-2ATI/OT, MCP73831T-2ATI_OT:SOT95P280X145-5N
- D2: value BLUE -> BLUE-0402; device SparkFun-LED:LED-0603 -> OPL_Optoelectronics:LED-0402
- R14: value 1k -> (none); device SparkFun-Resistors:0603 -> SparkFun-Resistors:0402
- moved RGB48 487.7 mm to (81.3, 82.5)
- moved RGB47 480.1 mm to (74.9, 82.5)
- moved RGB46 472.5 mm to (68.6, 82.5)
- moved RGB45 465.0 mm to (62.2, 82.5)
- moved RGB44 457.6 mm to (55.9, 82.5)
- moved RGB43 450.2 mm to (49.5, 82.5)
- moved Q1 445.0 mm to (36.5, 42.7), flipped to the bottom, turned to 270 degrees
- moved RGB42 442.8 mm to (43.2, 82.5)
- moved RGB41 435.6 mm to (36.8, 82.5)
- moved RGB40 428.4 mm to (30.5, 82.5)
- moved RGB39 421.2 mm to (24.1, 82.5)
- moved RGB38 414.2 mm to (17.8, 82.5)
- moved RGB37 407.2 mm to (11.4, 82.5)
- moved RGB36 389.4 mm to (81.3, 57.1)
- moved RGB35 381.5 mm to (74.9, 57.1)
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Connections:
- removed net G1: Q1.4
- removed net G2: Q1.2
- removed net XOUT: R14.1, U1.21
- new net DI_NEOPIXEL: LED1.3, U1.32
- new net DO1: LED1.1, LED2.3
- new net DO10: LED10.1, LED11.3
- new net DO11: LED11.1, LED12.3
- new net DO2: LED2.1, LED3.3
- new net DO3: LED3.1, LED4.3
- new net DO4: LED4.1, LED5.3
- new net DO5: LED5.1, LED6.3
- new net DO6: LED6.1, LED7.3
- new net DO7: LED7.1, LED8.3
- new net DO8: LED8.1, LED9.3
- new net DO9: LED10.3, LED9.1
- new net INT1: U1.27, U2.4
- new net INT2: U1.28, U2.9
- new net INTB: IC2.37, R18.1, U1.31
- new net N$10: IC2.30, R15.1
- new net N$11: J2.2, Q2.3
- new net N$12: D1.-, R12.2
- new net N$13: R12.1, U4.1
- new net N$14: C22.1, J1.A4_B9, J1.B4_A9, L2.1
- new net N$15: R13.2, U4.5
- new net N$16: D4.+, R19.1
- new net N$17: JP1.2, R19.2
- new net N$18: IC2.39, R16.2
- new net N$4: C20.2, Q1.3, R14.1
- new net N$5: J1.A5, R8.2
- new net N$6: R14.2, U1.21
- new net N$8: J1.B5, R9.2
- new net N$9: S3.1, S3.2, U1.30
- new net SDB: IC2.38, R17.2, U1.29
- new net SDO: R7.2, U1.18, U2.1
- new net VIN: C16.2, C24.2, C25.1, C26.2, C27.1, C28.2, C29.1, C42.+, D3.-, IC2.19, IC2.26, IC2.31, SW1.2, U3.1, U3.3
- new net V_BATT: C18.2, Q2.2, SW1.1, U4.3
- new net V_USB: C17.2, C23.1, D1.+, D3.+, L2.2, Q2.1, R11.2, U4.4
- net !BOOT: now also R4.2
- net 3.3V: now also C13.1, C14.1, C15.2, C19.1, C30.2, C31.2, C32.2, C33.2, C34.2, C35.2, C36.2, C37.2, C38.2, C39.2, C40.2, C41.2, IC2.32, JP1.1, LED1.4, LED10.4, LED11.4, LED12.4, LED2.4, LED3.4, LED4.4, LED5.4, LED6.4, LED7.4, LED8.4, LED9.4, MK1.5, R18.2, R3.2, R5.2, R6.2, U2.12, U2.5, U2.8, U3.5
- net CLK: now also MK1.4
- net CS1: now also IC2.15
- net CS10: now also IC2.25
- net CS11: now also IC2.27
- net CS12: now also IC2.28
- net CS2: now also IC2.16
- net CS3: now also IC2.17
- net CS4: now also IC2.18
- net CS5: now also IC2.20
- net CS6: now also IC2.21
- net CS7: now also IC2.22
- net CS8: now also IC2.23
- net CS9: now also IC2.24
- net DATA: now also MK1.1
- net GND: now also C13.2, C14.2, C15.1, C16.1, C17.1, C18.1, C19.2, C20.1, C21.1, C22.2, C23.2, C24.1, C25.2, C26.1, C27.2, C28.1, C29.2, C30.1, C31.1, C32.1, C33.1, C34.1, C35.1, C36.1, C37.1, C38.1, C39.1, C40.1, C41.1, C42.-, D2.-, D4.-, IC2.36, J1.A1_B12, J1.B1_A12, J2.1, LED1.2, LED10.2, LED11.2, LED12.2, LED2.2, LED3.2, LED4.2, LED5.2, LED6.2, LED7.2, LED8.2, LED9.2, MK1.2, MK1.3, Q1.2, Q1.4, R11.1, R13.1, R15.2, R16.1, R17.1, R7.1, R8.1, R9.1, S3.3, S3.4, SW1.S1, SW1.S2, SW1.S3, SW1.S4, U2.6, U2.7, U3.2, U4.2; no longer C20.2, C21.2, D2.C
- net N$1: now also D2.+; no longer D2.A
- net QSPI_CS: now also IC1.1, R3.1, R4.1
- net QSPI_SCLK: now also IC1.6
- net QSPI_SD0: now also IC1.5
- net QSPI_SD1: now also IC1.2
- net QSPI_SD2: now also IC1.3
- net QSPI_SD3: now also IC1.7
- net SCL: now also IC2.35, R5.1, U2.13
- net SDA: now also IC2.34, R6.1, U2.14
- net SW01: now also IC2.1
- net SW02: now also IC2.2
- net SW03: now also IC2.3
- net SW04: now also IC2.5
- net SW05: now also IC2.6
- net SW06: now also IC2.7
- net SW07: now also IC2.8
- net SW08: now also IC2.9
- net SW09: now also IC2.10
- net SW10: now also IC2.12
- net SW11: now also IC2.13
- net SW12: now also IC2.14
- net USB_N: now also J1.A7, J1.B7
- net USB_P: now also J1.A6, J1.B6
- net XIN: now also C21.2, Q1.1; no longer C20.1
Routing:
- net SW03: track 0.00 -> 101.0 mm, vias 0 -> 12
- net SW02: track 0.00 -> 100.1 mm, vias 0 -> 12
- net SW07: track 0.00 -> 98.0 mm, vias 0 -> 12
- net SW09: track 0.00 -> 97.8 mm, vias 0 -> 12
- net SW08: track 0.00 -> 96.7 mm, vias 0 -> 12
- net SW04: track 0.00 -> 92.8 mm, vias 0 -> 12
- net SW06: track 0.00 -> 92.0 mm, vias 0 -> 12
- net SW12: track 0.00 -> 91.8 mm, vias 0 -> 12
- net SW10: track 0.00 -> 91.6 mm, vias 0 -> 12
- net CS6: track 0.00 -> 91.2 mm
- net SW11: track 0.00 -> 91.0 mm, vias 0 -> 12
- net SW05: track 0.00 -> 90.3 mm, vias 0 -> 12
- net SW01: track 0.00 -> 88.8 mm, vias 0 -> 12
- net CS12: track 0.00 -> 84.6 mm
- net CS8: track 0.00 -> 83.0 mm
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- added copper zone on layer 15, net 3.3V
- added copper zone on layer 1, net GND
- added copper zone on layer 15, net GND
- added copper zone on layer 16, net GND
- added copper zone on layer 2, net GND

Commit message: Board check-in
Parts:
- added C43: 0.1uF, SparkFun-Capacitors:0402
- C20, C21: value 27pf -> 33pf; device OPL_Capacitor:C0603 -> OPL_Capacitor:C0402
- R11: value 10k -> 10K; device SparkFun-Resistors:0603 -> SparkFun-Resistors:0402
- moved R16 1.79 mm to (9.80, 23.1)
- moved C8 1.49 mm to (24.5, 36.6)
- moved R3 0.88 mm to (2.80, 53.2)
- moved R4 0.77 mm to (4.37, 53.2)
- moved D2 0.72 mm to (23.5, 34.3)
- moved R10 0.70 mm to (23.0, 36.6)
- moved C13 0.56 mm to (-2.77, 24.0), turned to 270 degrees
- moved C14 0.52 mm to (-0.97, 31.0)
- moved C24 0.49 mm to (5.60, 10.7)
- moved C21 0.39 mm to (36.8, 45.2)
- moved C20 0.32 mm to (36.2, 39.9)
- moved C25 0.29 mm to (2.22, 10.5), turned to 270 degrees
- moved C12 0.20 mm to (-10.3, 53.2)
- turned R9 to 180 degrees
Connections:
- net GND: now also C43.1, H1.P$1, H2.P$1, H3.P$1, H4.P$1, H5.P$1, H6.P$1, H7.P$1, H8.P$1
- net SDB: now also C43.2
Routing:
- net 3.3V: track 78.8 -> 247.3 mm, vias 7 -> 29
- net SW01: track 88.8 -> 232.6 mm, vias 12 -> 13
- net SW02: track 100.1 -> 241.4 mm, vias 12 -> 13
- net SW03: track 101.0 -> 240.2 mm, vias 12 -> 13
- net SW04: track 92.8 -> 210.4 mm, vias 12 -> 13
- net SW05: track 90.3 -> 207.7 mm, vias 12 -> 13
- net SW06: track 92.0 -> 209.2 mm, vias 12 -> 13
- net CS12: track 84.6 -> 191.0 mm, vias 0 -> 1
- net CS11: track 78.3 -> 176.0 mm, vias 0 -> 1
- net DI_NEOPIXEL: track 0.00 -> 91.5 mm, vias 0 -> 3
- net CS10: track 77.9 -> 167.0 mm, vias 0 -> 1
- net CS9: track 83.0 -> 164.0 mm, vias 0 -> 1
- net CS8: track 83.0 -> 156.4 mm, vias 0 -> 1
- net VIN: track 0.00 -> 71.3 mm, vias 0 -> 4
- net CS7: track 77.9 -> 143.1 mm, vias 0 -> 1
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