File: piboard.sch (EAGLE design)
At the start: 79 parts, among them IC1 IS25LP256D-JLLE-TR, IC2 IS31FL3737-QFLS4-TR, U1 RP2040, Y1 ABLS-12.000MHZ-B4-T

Commit message: Daily check-in
Parts:
- removed Y1: ABLS-12.000MHZ-B4-T, ABLS-12.000MHZ-B4-T:ABLS-12.000MHZ-B4-T
- added Q1: (no value), adafruit:XTAL-4-3225
Connections:
- removed net XOUT_R: C21.1, R14.2, Y1.1
- new net SW01: RGB37.G_C, RGB38.G_C, RGB39.G_C, RGB40.G_C, RGB41.G_C, RGB42.G_C, RGB43.G_C, RGB44.G_C, RGB45.G_C, RGB46.G_C, RGB47.G_C, RGB48.G_C
- new net SW02: RGB37.R_C, RGB38.R_C, RGB39.R_C, RGB40.R_C, RGB41.R_C, RGB42.R_C, RGB43.R_C, RGB44.R_C, RGB45.R_C, RGB46.R_C, RGB47.R_C, RGB48.R_C
- new net SW03: RGB37.B_C, RGB38.B_C, RGB39.B_C, RGB40.B_C, RGB41.B_C, RGB42.B_C, RGB43.B_C, RGB44.B_C, RGB45.B_C, RGB46.B_C, RGB47.B_C, RGB48.B_C
- new net SW04: RGB25.G_C, RGB26.G_C, RGB27.G_C, RGB28.G_C, RGB29.G_C, RGB30.G_C, RGB31.G_C, RGB32.G_C, RGB33.G_C, RGB34.G_C, RGB35.G_C, RGB36.G_C
- new net SW05: RGB25.R_C, RGB26.R_C, RGB27.R_C, RGB28.R_C, RGB29.R_C, RGB30.R_C, RGB31.R_C, RGB32.R_C, RGB33.R_C, RGB34.R_C, RGB35.R_C, RGB36.R_C
- new net SW06: RGB25.B_C, RGB26.B_C, RGB27.B_C, RGB28.B_C, RGB29.B_C, RGB30.B_C, RGB31.B_C, RGB32.B_C, RGB33.B_C, RGB34.B_C, RGB35.B_C, RGB36.B_C
- new net SW07: RGB13.G_C, RGB14.G_C, RGB15.G_C, RGB16.G_C, RGB17.G_C, RGB18.G_C, RGB19.G_C, RGB20.G_C, RGB21.G_C, RGB22.G_C, RGB23.G_C, RGB24.G_C
- new net SW08: RGB13.R_C, RGB14.R_C, RGB15.R_C, RGB16.R_C, RGB17.R_C, RGB18.R_C, RGB19.R_C, RGB20.R_C, RGB21.R_C, RGB22.R_C, RGB23.R_C, RGB24.R_C
- new net SW09: RGB13.B_C, RGB14.B_C, RGB15.B_C, RGB16.B_C, RGB17.B_C, RGB18.B_C, RGB19.B_C, RGB20.B_C, RGB21.B_C, RGB22.B_C, RGB23.B_C, RGB24.B_C
- net GND: now also IC2.EP, IC2.GND, IC2.PGND_1, IC2.PGND_2
- net XIN: no longer Y1.2

Commit message: update
Parts:
- added C13, C14, C22, C23, C25, C27, C29: 0.1uF, SparkFun-Capacitors:0.1UF-0402-16V-10%
- added C15, C16: 10uF, OPL_Capacitor:CERAMIC-10UF-6.3V-20%-X5R(0402)
- added C17, C18: 4.7uF, OPL_Capacitor:CERAMIC-4.7UF-6.3V-20%-X5R(0402)
- added C19, C24, C26, C28: 470nF 50V, OPL_Capacitor:CERAMIC-390PF-50V-10%-X7R(0402)
- added C30, C31, C32, C33, C34, C35, C36, C37, C38, C39, C40, C41: 100nf, OPL_Capacitor:CERAMIC-100NF-25V-10%-X7R(0402)
- added C42: 22uF, OPL_Capacitor:TANTALUM-SMD-22UF-10V(AVX-A)
- added D1: BLUE-0402, OPL_Optoelectronics:SMD-LED-CLEAR-BLUE(0402)
- added D3: 20V-1A, OPL_Discrete_Semiconductor:SMD-DIODE-SCHOTTKY-20V-1A(SOD-123)
- added D4: RED-0402, OPL_Optoelectronics:SMD-LED-CLEAR-BLUE(0402)
- added H1, H2, H3, H4, H5, H6, H7, H8: M25, M25:M25
- added J1: TYPE-C-31-M-12, TYPE-C-31-M-12:TYPE-C-31-M-12
- added J2: (no value), SparkFun-Connectors:JST_2MM_MALE
- added JP1: JUMPER-SMT_2_NO_SILK_ROUND, SparkFun-Jumpers:JUMPER-SMT_2_NO_SILK_ROUND
- added L2: 2.2nH, SparkFun-Coils:INDUCTOR-0402-3.9NH
- added LED1, LED10, LED11, LED12, LED2, LED3, LED4, LED5, LED6, LED7, LED8, LED9: WS2812B-2020, WS2812B-2020:WS2812B-2020
- added MK1: ICS-41350, ICS-41350:ICS-41350
- added Q2: 2.5A/30V/105mΩ, SparkFun-DiscreteSemi:MOSFET_PCH-DMG2307L
- added R11: 10k, SparkFun-Resistors:10KOHM-0603-1/10W-1%
- added R12: 470, SparkFun-Resistors:RESISTOR0402
- added R13: 2K, SparkFun-Resistors:RESISTOR0402
- added R15: 20K, SparkFun-Resistors:RESISTOR0402
- added R16, R17, R18: 100K, SparkFun-Resistors:100KOHM-0402-1/16W-1%
- added R19: 220, SparkFun-Resistors:RESISTOR0402
- added R3, R4, R7: 10K, SparkFun-Resistors:RESISTOR0402
- added R5, R6: 4.7K, SparkFun-Resistors:RESISTOR0402
- added R8, R9: 5.1K, SparkFun-Resistors:RESISTOR0402
- added S3: MOMENTARY-SWITCH-SPST-SMD-4.6X2.8MM, SparkFun-Switches:MOMENTARY-SWITCH-SPST-SMD-4.6X2.8MM
- added SW1: PCM12SMTR, PCM12SMTR:PCM12SMTR
- added U2: BMI270, BMI270:BMI270
- added U3: MIC5504-3.3YM5_TR, MIC5504-3.3YM5_TR:MIC5504-3.3YM5_TR
- added U4: MCP73831T-2ATI/OT, MCP73831T-2ATI_OT:MCP73831T-2ATI/OT
- D2: value BLUE -> BLUE-0402; device SparkFun-LED:LED-BLUE0603 -> OPL_Optoelectronics:SMD-LED-CLEAR-BLUE(0402)
- R14: value 1k -> (none); device SparkFun-Resistors:1KOHM-0603-1/10W-1% -> SparkFun-Resistors:RESISTOR0402
Connections:
- removed net XOUT: R14.1, U1.XOUT
- new net DI_NEOPIXEL: LED1.DI, U1.GPIO21
- new net DO1: LED1.DO, LED2.DI
- new net DO10: LED10.DO, LED11.DI
- new net DO11: LED11.DO, LED12.DI
- new net DO2: LED2.DO, LED3.DI
- new net DO3: LED3.DO, LED4.DI
- new net DO4: LED4.DO, LED5.DI
- new net DO5: LED5.DO, LED6.DI
- new net DO6: LED6.DO, LED7.DI
- new net DO7: LED7.DO, LED8.DI
- new net DO8: LED8.DO, LED9.DI
- new net DO9: LED10.DI, LED9.DO
- new net INT1: U1.GPIO16, U2.INT1
- new net INT2: U1.GPIO17, U2.INT2
- new net INTB: IC2.INTB, R18.1, U1.GPIO20
- new net N$10: IC2.RSET, R15.1
- new net N$11: J2.+, Q2.D
- new net N$12: D1.-, R12.2
- new net N$13: R12.1, U4.STAT
- new net N$14: C22.1, J1.VBUS, L2.1
- new net N$15: R13.2, U4.PROG
- new net N$16: D4.+, R19.1
- new net N$17: JP1.2, R19.2
- new net N$18: IC2.IICRST, R16.2
- new net N$4: C20.2, Q1.X2, R14.1
- new net N$5: J1.CC1, R8.2
- new net N$6: R14.2, U1.XOUT
- new net N$8: J1.CC2, R9.2
- new net N$9: S3.1, U1.GPIO19
- new net SDB: IC2.SDB, R17.2, U1.GPIO18
- new net SDO: R7.2, U1.GPIO15, U2.SDO
- new net VIN: C16.2, C24.2, C25.1, C26.2, C27.1, C28.2, C29.1, C42.+, D3.-, IC2.PVCC_1, IC2.PVCC_2, IC2.VCC, SW1.2, U3.EN, U3.VIN
- new net V_BATT: C18.2, Q2.S, SW1.1, U4.VBAT
- new net V_USB: C17.2, C23.1, D1.+, D3.+, L2.2, Q2.G, R11.2, U4.VDD
- net !BOOT: now also R4.2
- net 3.3V: now also C13.1, C14.1, C15.2, C19.1, C30.2, C31.2, C32.2, C33.2, C34.2, C35.2, C36.2, C37.2, C38.2, C39.2, C40.2, C41.2, IC2.VIO, JP1.1, LED1.VDD, LED10.VDD, LED11.VDD, LED12.VDD, LED2.VDD, LED3.VDD, LED4.VDD, LED5.VDD, LED6.VDD, LED7.VDD, LED8.VDD, LED9.VDD, MK1.VDD, R18.2, R3.2, R5.2, R6.2, U2.CSB, U2.VDD, U2.VDDIO, U3.VOUT
- net CLK: now also MK1.CLK
- net CS1: now also IC2.CS1
- net CS10: now also IC2.CS10
- net CS11: now also IC2.CS11
- net CS12: now also IC2.CS12
- net CS2: now also IC2.CS2
- net CS3: now also IC2.CS3
- net CS4: now also IC2.CS4
- net CS5: now also IC2.CS5
- net CS6: now also IC2.CS6
- net CS7: now also IC2.CS7
- net CS8: now also IC2.CS8
- net CS9: now also IC2.CS9
- net DATA: now also MK1.DATA
- net GND: now also C13.2, C14.2, C15.1, C16.1, C17.1, C18.1, C19.2, C20.1, C21.1, C22.2, C23.2, C24.1, C25.2, C26.1, C27.2, C28.1, C29.2, C30.1, C31.1, C32.1, C33.1, C34.1, C35.1, C36.1, C37.1, C38.1, C39.1, C40.1, C41.1, C42.-, D2.-, D4.-, IC2.ADDR, J1.GND, J2.-, LED1.VSS, LED10.VSS, LED11.VSS, LED12.VSS, LED2.VSS, LED3.VSS, LED4.VSS, LED5.VSS, LED6.VSS, LED7.VSS, LED8.VSS, LED9.VSS, MK1.GND, MK1.SELECT, Q1.G1, Q1.G2, R11.1, R13.1, R15.2, R16.1, R17.1, R7.1, R8.1, R9.1, S3.2, SW1.SHIELD, U2.GND, U2.GNDIO, U3.GND, U4.VSS; no longer C20.2, C21.2, D2.C
- net N$1: now also D2.+; no longer D2.A
- net QSPI_CS: now also IC1.CE#, R3.1, R4.1
- net QSPI_SCLK: now also IC1.SCK
- net QSPI_SD0: now also IC1.SI_(IO0)
- net QSPI_SD1: now also IC1.SO_(IO1)
- net QSPI_SD2: now also IC1.WP#_(IO2)
- net QSPI_SD3: now also IC1.HOLD#
- net SCL: now also IC2.SCL, R5.1, U2.SCX
- net SDA: now also IC2.SDA, R6.1, U2.SDX
- net SW01: now also IC2.SW1
- net SW02: now also IC2.SW2
- net SW03: now also IC2.SW3
- net SW04: now also IC2.SW4
- net SW05: now also IC2.SW5
- net SW06: now also IC2.SW6
- net SW07: now also IC2.SW7
- net SW08: now also IC2.SW8
- net SW09: now also IC2.SW9
- net SW10: now also IC2.SW10
- net SW11: now also IC2.SW11
- net SW12: now also IC2.SW12
- net USB_N: now also J1.DN1, J1.DN2
- net USB_P: now also J1.DP1, J1.DP2
- net XIN: now also C21.2, Q1.X1; no longer C20.1
Other:
- note added: "USB"

Commit message: Board check-in
Parts:
- added C43: 0.1uF, SparkFun-Capacitors:0.1UF-0402-16V-10%
- C20, C21: value 27pf -> 33pf; device OPL_Capacitor:CERAMIC-27PF-50V-5%-NPO(0603) -> OPL_Capacitor:CERAMIC-33PF-50V-5%-NPO(0402)
- R11: value 10k -> 10K; device SparkFun-Resistors:10KOHM-0603-1/10W-1% -> SparkFun-Resistors:RESISTOR0402
Connections:
- net GND: now also C43.1, H1.P$1, H2.P$1, H3.P$1, H4.P$1, H5.P$1, H6.P$1, H7.P$1, H8.P$1
- net SDB: now also C43.2
